File: pico-calc2.kicad_pcb (KiCad board)
At the start: 2 copper layers, 2 parts, among them U1 Pimoroni_Pico_LiPo_2_XL_W

Commit message: oijojojaf'skjdkfjalsdklfjsa
asdfasdf
Parts:
- added U2: TPS60230, Package_DFN_QFN:Texas_RGV0016A_VQFN-16-1EP_4x4mm_P0.65mm_EP2.1x2.1mm, F.Cu at (62.7, 15.7)
- DS1: footprint Library:HRS_FH12-45S-0.5SH_55_ -> Library:CONN_S-45S-0.5SH55
- moved DS1 123.6 mm to (45.0, 10.0)
- moved U1 33.8 mm to (64.4, 39.2), turned to -90 degrees
Connections:
- DS1 pad 1: unconnected-(DS1-GND-Pad1) -> GND
- DS1 pad 10: unconnected-(DS1-HSYNC-Pad10) -> GND
- DS1 pad 11: unconnected-(DS1-DOTCLK-Pad11) -> GND
- DS1 pad 12: unconnected-(DS1-ENABLE-Pad12) -> GND
- DS1 pad 13: unconnected-(DS1-RD-Pad13) -> /DISP_RD
- DS1 pad 14: unconnected-(DS1-WR_(SPI-RS)-Pad14) -> /DISP_WR
- DS1 pad 15: unconnected-(DS1-RS_(SPI-SCL)-Pad15) -> /DISP_RS
- DS1 pad 16: unconnected-(DS1-CS-Pad16) -> /DISP_CS
- DS1 pad 17: unconnected-(DS1-RESET-Pad17) -> /DISP_RESET
- DS1 pad 18: unconnected-(DS1-DB0-Pad18) -> /DISP_DB0
- DS1 pad 19: unconnected-(DS1-DB1-Pad19) -> /DISP_DB1
- DS1 pad 2: unconnected-(DS1-GND-Pad2) -> GND
- DS1 pad 20: unconnected-(DS1-DB2-Pad20) -> /DISP_DB2
- DS1 pad 21: unconnected-(DS1-DB3-Pad21) -> /DISP_DB3
- DS1 pad 22: unconnected-(DS1-DB4-Pad22) -> /DISP_DB4
- DS1 pad 23: unconnected-(DS1-DB5-Pad23) -> /DISP_DB5
- DS1 pad 24: unconnected-(DS1-DB6-Pad24) -> /DISP_DB6
- DS1 pad 25: unconnected-(DS1-DB7-Pad25) -> /DISP_DB7
- DS1 pad 26: unconnected-(DS1-DB8-Pad26) -> /DISP_DB8
- DS1 pad 27: unconnected-(DS1-DB9-Pad27) -> GND
- DS1 pad 28: unconnected-(DS1-DB10-Pad28) -> GND
- DS1 pad 29: unconnected-(DS1-DB11-Pad29) -> GND
- DS1 pad 3: unconnected-(DS1-IOVCC-Pad3) -> +3V3
- DS1 pad 30: unconnected-(DS1-DB12-Pad30) -> GND
- DS1 pad 31: unconnected-(DS1-DB13-Pad31) -> GND
- DS1 pad 32: unconnected-(DS1-DB14-Pad32) -> GND
- DS1 pad 33: unconnected-(DS1-DB15-Pad33) -> GND
- DS1 pad 34: unconnected-(DS1-DB16-Pad34) -> GND
- DS1 pad 35: unconnected-(DS1-DB17-Pad35) -> GND
- DS1 pad 36: unconnected-(DS1-LEDK1-Pad36) -> /LEDK1
- DS1 pad 37: unconnected-(DS1-LEDK2-Pad37) -> /LEDK2
- DS1 pad 38: unconnected-(DS1-LEDK3-Pad38) -> /LEDK3
- DS1 pad 39: unconnected-(DS1-LEDK4-Pad39) -> /LEDK4
- DS1 pad 4: unconnected-(DS1-VCI-Pad4) -> +3V3
- DS1 pad 40: unconnected-(DS1-LEDA-Pad40) -> /LEDA
- DS1 pad 45: unconnected-(DS1-GND-Pad45) -> GND
- DS1 pad 5: unconnected-(DS1-IM3-Pad5) -> GND
- DS1 pad 6: unconnected-(DS1-IM2-Pad6) -> GND
- DS1 pad 7: unconnected-(DS1-IM0-Pad7) -> +3V3
- DS1 pad 8: unconnected-(DS1-SDA-Pad8) -> GND
- DS1 pad 9: unconnected-(DS1-VSYNC-Pad9) -> GND
- U1 pad 11: unconnected-(U1-GP8-Pad11) -> /BRIGHTNESS
- U1 pad 12: unconnected-(U1-GP9-Pad12) -> /DISP_DB8
- U1 pad 13: unconnected-(U1-GND-Pad13) -> Net-(U1-GND-Pad13)
- U1 pad 14: unconnected-(U1-GP10-Pad14) -> /DISP_DB7
- U1 pad 15: unconnected-(U1-GP11-Pad15) -> /DISP_DB6
- U1 pad 16: unconnected-(U1-GP12-Pad16) -> /DISP_DB5
- U1 pad 17: unconnected-(U1-GP13-Pad17) -> /DISP_DB4
- U1 pad 18: unconnected-(U1-GND-Pad18) -> Net-(U1-GND-Pad13)
- U1 pad 19: unconnected-(U1-GP14-Pad19) -> /DISP_DB3
- U1 pad 20: unconnected-(U1-GP15-Pad20) -> /DISP_DB2
- U1 pad 23: unconnected-(U1-GND-Pad23) -> Net-(U1-GND-Pad13)
- U1 pad 28: unconnected-(U1-GND-Pad28) -> Net-(U1-GND-Pad13)
- U1 pad 3: unconnected-(U1-GND-Pad3) -> Net-(U1-GND-Pad13)
- U1 pad 33: unconnected-(U1-GND-Pad33) -> Net-(U1-GND-Pad13)
- U1 pad 36: unconnected-(U1-3V3-Pad36) -> +3V3
- U1 pad 38: unconnected-(U1-GND-Pad38) -> Net-(U1-GND-Pad13)
- U1 pad 41: unconnected-(U1-3V3-Pad41) -> +3V3
- U1 pad 42: unconnected-(U1-GP31-Pad42) -> /DISP_DB1
- U1 pad 43: unconnected-(U1-GND-Pad43) -> Net-(U1-GND-Pad13)
- U1 pad 44: unconnected-(U1-GP32-Pad44) -> /DISP_DB0
- U1 pad 45: unconnected-(U1-GP33-Pad45) -> /DISP_RESET
- U1 pad 46: unconnected-(U1-GP34-Pad46) -> /DISP_CS
- U1 pad 47: unconnected-(U1-GP35-Pad47) -> /DISP_RS
- U1 pad 48: unconnected-(U1-GND-Pad48) -> Net-(U1-GND-Pad13)
- U1 pad 49: unconnected-(U1-GP36-Pad49) -> /DISP_WR
- U1 pad 50: unconnected-(U1-GP37-Pad50) -> /DISP_RD
- U1 pad 53: unconnected-(U1-GND-Pad53) -> Net-(U1-GND-Pad13)
- U1 pad 58: unconnected-(U1-GND-Pad58) -> Net-(U1-GND-Pad13)
- U1 pad 8: unconnected-(U1-GND-Pad8) -> Net-(U1-GND-Pad13)
Routing:
- net /LEDA: track 0.00 -> 12.0 mm, vias 0 -> 2
- net /LEDK4: track 0.00 -> 11.8 mm
- net /LEDK1: track 0.00 -> 11.0 mm
- net /LEDK3: track 0.00 -> 10.6 mm
- net /LEDK2: track 0.00 -> 10.3 mm
- net GND: track 0.00 -> 3.99 mm
Other:
- board outline added: 90 x 100 mm
