File: pico-calc2.kicad_sch (KiCad schematic)
At the start: 63 parts, among them SW1 SW_Push_45deg, SW10 SW_Push_45deg, SW11 SW_Push_45deg, SW12 SW_Push_45deg, SW13 SW_Push_45deg, SW14 SW_Push_45deg, SW15 SW_Push_45deg, SW16 SW_Push_45deg, SW17 SW_Push_45deg, SW18 SW_Push_45deg, SW19 SW_Push_45deg, SW2 SW_Push_45deg, SW20 SW_Push_45deg, SW21 SW_Push_45deg, SW22 SW_Push_45deg, SW23 SW_Push_45deg, SW24 SW_Push_45deg, SW25 SW_Push_45deg, SW26 SW_Push_45deg, SW27 SW_Push_45deg, SW28 SW_Push_45deg, SW29 SW_Push_45deg, SW3 SW_Push_45deg, SW30 SW_Push_45deg, SW31 SW_Push_45deg, SW32 SW_Push_45deg, SW33 SW_Push_45deg, SW34 SW_Push_45deg, SW35 SW_Push_45deg, SW36 SW_Push_45deg, SW37 SW_Push_45deg, SW38 SW_Push_45deg, SW39 SW_Push_45deg, SW4 SW_Push_45deg, SW40 SW_Push_45deg, SW41 SW_Push_45deg, SW42 SW_Push_45deg, SW43 SW_Push_45deg, SW44 SW_Push_45deg, SW45 SW_Push_45deg, SW46 SW_Push_45deg, SW47 SW_Push_45deg, SW48 SW_Push_45deg, SW49 SW_Push_45deg, SW5 SW_Push_45deg, SW50 SW_Push_45deg, SW51 SW_Push_45deg, SW52 SW_Push_45deg, SW53 SW_Push_45deg, SW54 SW_Push_45deg, SW55 SW_Push_45deg, SW56 SW_Push_45deg, SW57 SW_Push_45deg, SW58 SW_Push_45deg, SW59 SW_Push_45deg, SW6 SW_Push_45deg, SW60 SW_Push_45deg, SW7 SW_Push_45deg, SW8 SW_Push_45deg, SW9 SW_Push_45deg, U1 Pimoroni_Pico_LiPo_2_XL_W, U2 TPS60230

Commit message: oijojojaf'skjdkfjalsdklfjsa
asdfasdf
Parts:
- added C1, C2: .47u, symbol Device:C
- added C4, C5: 1u, symbol Device:C
- added R1: R, symbol Device:R
- DS1: footprint Library:HRS_FH12-45S-0.5SH_55_ -> Library:CONN_S-45S-0.5SH55
Connections:
- net GND: now reaches DS1.1 (GND)
- net GND: now also DS1.10 (HSYNC), DS1.11 (DOTCLK), DS1.12 (ENABLE), DS1.2 (GND), DS1.27 (DB9), DS1.28 (DB10), DS1.29 (DB11), DS1.30 (DB12), DS1.31 (DB13), DS1.32 (DB14), DS1.33 (DB15), DS1.34 (DB16), DS1.35 (DB17), DS1.45 (GND), DS1.5 (IM3), DS1.6 (IM1), DS1.8 (SDA), DS1.9 (VSYNC), U2.14 (GND), U2.17 (PAD), U2.7 (PGND), C4.2, C5.2, R1.2
- net DISP_RD: now reaches DS1.13 (RD)
- net DISP_RD: now also U1.50 (GP37)
- net DISP_WR: now reaches DS1.14 (WR_(SPI-RS))
- net DISP_WR: now also U1.49 (GP36)
- net DISP_RS: now reaches DS1.15 (RS_(SPI-SCL))
- net DISP_RS: now also U1.47 (GP35)
- net DISP_CS: now reaches DS1.16 (CS)
- net DISP_CS: now also U1.46 (GP34)
- net DISP_RESET: now reaches DS1.17 (RESET)
- net DISP_RESET: now also U1.45 (GP33)
- net DISP_DB0: now reaches DS1.18 (DB0)
- net DISP_DB0: now also U1.44 (GP32)
- net DISP_DB1: now reaches DS1.19 (DB1)
- net DISP_DB1: now also U1.42 (GP31)
- net DISP_DB2: now reaches DS1.20 (DB2)
- net DISP_DB2: now also U1.20 (GP15)
- net DISP_DB3: now reaches DS1.21 (DB3)
- net DISP_DB3: now also U1.19 (GP14)
- net DISP_DB4: now reaches DS1.22 (DB4)
- net DISP_DB4: now also U1.17 (GP13)
- net DISP_DB5: now reaches DS1.23 (DB5)
- net DISP_DB5: now also U1.16 (GP12)
- net DISP_DB6: now reaches DS1.24 (DB6)
- net DISP_DB6: now also U1.15 (GP11)
- net DISP_DB7: now reaches DS1.25 (DB7)
- net DISP_DB7: now also U1.14 (GP10)
- net DISP_DB8: now reaches DS1.26 (DB8)
- net DISP_DB8: now also U1.12 (GP9)
- net +3V3: now reaches DS1.3 (VCC)
- net +3V3: now also DS1.4 (VCC), DS1.7 (IM0), U1.36 (3V3), U2.13 (VIN), C4.1
- net LEDK1: now reaches DS1.36 (LEDK1)
- net LEDK1: now also U2.6 (D1)
- net LEDK2: now reaches DS1.37 (LEDK2)
- net LEDK2: now also U2.5 (D2)
- net LEDK3: now reaches DS1.38 (LEDK3)
- net LEDK3: now also U2.4 (D3)
- net LEDK4: now reaches DS1.39 (LEDK4)
- net LEDK4: now also U2.3 (D4)
- net LEDA: now reaches DS1.40 (LEDA)
- net LEDA: now also U2.8 (VOUT), C5.1
- net BRIGHTNESS: now reaches U1.11 (GP8)
- net BRIGHTNESS: now also U2.15 (EN1), U2.16 (EN2)
- net at U2.1 (ISET): now also R1.1
- net at U2.10 (C1-): now also C1.1
- net at U2.11 (C1+): now also C1.2
- net at U2.12 (C2-): now also C2.1
- net at U2.9 (C2+): now also C2.2
- no-connect marks 0 -> 5
Other:
- note added: "R_{ISET} = 260 * (V_{ISET}/I_{LED}) ~ 7.8k"
- moved on the sheet: DS1, U1, U2
